Commit message: add pointcloud to laserscan

File: robot_description/urdf/my_robot_urdf/my_robot_core.xacro (robot description, xacro)
@@ -5,5 +5,5 @@
   <link name="base_link"></link>
   <link name="chassi">
-    <xacro:inertial_box mass="1" x="${lenght_robot}" y="${width_robot}" z="${height_robot}">
+    <xacro:inertial_box mass="0.3" x="${lenght_robot}" y="${width_robot}" z="${height_robot}">
       <origin xyz="0.0 0.0 ${height_robot/2}" />
     </xacro:inertial_box>
@@ -31,5 +31,5 @@
   </joint>
   <link name="wheel_left">
-    <xacro:inertial_cylinder mass="0.25" radius="${wheel_radius}" length="${wheel_length}">
+    <xacro:inertial_cylinder mass="0.4" radius="${wheel_radius}" length="${wheel_length}">
       <origin xyz="0.0 ${wheel_length/2} 0.0" />
     </xacro:inertial_cylinder>
@@ -58,5 +58,5 @@
   </joint>
   <link name="wheel_right">
-    <xacro:inertial_cylinder mass="0.25" radius="${wheel_radius}" length="${wheel_length}">
+    <xacro:inertial_cylinder mass="0.4" radius="${wheel_radius}" length="${wheel_length}">
       <origin xyz="0.0 ${wheel_length/2} 0.0" />
     </xacro:inertial_cylinder>
@@ -84,5 +84,31 @@
     <axis xyz="0.0 1 0.0" />
   </joint>
-  <!-- ROLING WHEEL -->
+    <!-- CASTER WHEEL LINK -->
+    <joint name="caster_wheel_joint" type="fixed">
+        <parent link="chassi"/>
+        <child link="caster_wheel"/>
+        <origin xyz="${caster_wheel_offset_x} 0 ${caster_wheel_offset_z}"/>
+    </joint>
+    <link name="caster_wheel">
+        <visual>
+            <geometry>
+                <sphere radius="${caster_wheel_radius}"/>
+            </geometry>
+            <material name="white"/>
+        </visual>
+        <collision>
+            <geometry>
+                <sphere radius="${caster_wheel_radius}"/>
+            </geometry>
+        </collision>
+        <xacro:inertial_sphere mass="${caster_wheel_mass}" radius="${caster_wheel_radius}">
+            <origin xyz="0 0 0" rpy="0 0 0"/>
+        </xacro:inertial_sphere>
+    </link>
+    <gazebo reference="caster_wheel">
+        <material>Gazebo/White</material>
+        <mu1 value="0.001"/>
+        <mu2 value="0.001"/>
+    </gazebo>
   <!-- DEPTH CAMERA -->
   <link name="base_depth_camera">

File: robot_description/urdf/my_robot_urdf/my_robot_property.xacro (robot description, xacro)
@@ -8,3 +8,7 @@
   <xacro:property name="wheel_length" value="0.03" />
   <xacro:property name="wheel_offset_x" value="0.1" />
+  <xacro:property name="caster_wheel_radius" value="${wheel_radius}"/>
+  <xacro:property name="caster_wheel_mass" value="0.8"/>
+  <xacro:property name="caster_wheel_offset_x" value="-0.1"/>
+  <xacro:property name="caster_wheel_offset_z" value="0"/>
 </robot>
